File: PCB/Projects/Main Board/Latte_Main_Board.kicad_pcb (KiCad board)
At the start: 4 copper layers, 114 x 50.5 mm, 113 parts, among them J1 SM02B-SURS-TF_LF__SN_, J2 SM02B-SURS-TF_LF__SN_, J3 Molex 505110-0892, J4 Molex 505110-0592, J5 Molex 505110-0892, J6 Molex 505110-0592, J8 Conn_01x04_Pin, J9 Molex 505110-1792, Q1 MMBT2222A, Q2 MMBT2222A, SW1 SW_Push, SW2 SW_Push, SW3 SW_Push, SW4 SW_Push, SW5 SW_Push, SW6 SW_Push, SW7 SW_Push, SW8 SW_Push, U1 HAL4395, U10 HAL4395, U11 HAL4395, U2 RP2350_80QFN, U3 HAL4395, U4 ST_LSM6, U5 ST_LSM6, U6 HAL4395, U7 HAL4395, U8 HAL4395, U9 HAL4395, Y1 ABM8-272-T3

Commit message: Routing updates
Parts:
- added C39: 4.7u, Capacitor_SMD:C_0402_1005Metric, B.Cu at (66.1, 49.9)
- added C40: 4.7u, Capacitor_SMD:C_0402_1005Metric, B.Cu at (65.2, 49.9)
- added R25: 100R, Resistor_SMD:R_0201_0603Metric, B.Cu at (52.9, 47.2)
- added R28: 100R, Resistor_SMD:R_0201_0603Metric, B.Cu at (27.9, 56.2)
- added R29: 100R, Resistor_SMD:R_0201_0603Metric, B.Cu at (124.5, 54.0)
- added R31: 100R, Resistor_SMD:R_0201_0603Metric, B.Cu at (91.8, 44.5)
- moved C5 183.6 mm to (118.7, 57.6), turned to -90 degrees
- moved C6 174.0 mm to (107.7, 66.7), turned to 90 degrees
- moved C3 171.7 mm to (107.7, 46.7), turned to 90 degrees
- moved C4 162.0 mm to (96.7, 56.7), turned to 90 degrees
- moved C8 119.5 mm to (55.2, 53.8), turned to 180 degrees
- moved C7 113.6 mm to (49.6, 49.1), turned to 90 degrees
- moved C18 110.3 mm to (44.7, 63.3), turned to -90 degrees
- moved C17 104.6 mm to (40.4, 53.8), turned to 180 degrees
- moved R2 32.7 mm to (91.8, 43.7), turned to 0 degrees
- moved R27 1.86 mm to (60.2, 46.5)
- moved R26 1.75 mm to (59.2, 48.4)
- moved L1 1.68 mm to (63.5, 49.9)
- moved R12 1.66 mm to (58.8, 47.2)
- moved R13 1.61 mm to (58.1, 47.2)
- moved R4 1.57 mm to (63.7, 48.2)
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Connections:
- C17 pad 1: Net-(U10-VCC) -> +3V3
- C18 pad 1: Net-(U11-VCC) -> +3V3
- C3 pad 1: Net-(U1-VCC) -> +3V3
- C4 pad 1: Net-(U3-VCC) -> +3V3
- C5 pad 1: Net-(U6-VCC) -> +3V3
- C6 pad 1: Net-(U7-VCC) -> +3V3
- C7 pad 1: Net-(U8-VCC) -> +3V3
- C8 pad 1: Net-(U9-VCC) -> +3V3
- J4 pad 2: TRIGGER_EN -> TRIGGER_EN_R
- J6 pad 2: TRIGGER_EN -> TRIGGER_EN_L
- R2 pad 1: Net-(U2-GPIO25) -> Net-(U2-GPIO26)
- R21 pad 1: Net-(U2-GPIO28) -> Net-(U2-GPIO29)
- R23 pad 1: Net-(U2-GPIO30) -> Net-(U2-GPIO39)
- R24 pad 1: Net-(U2-GPIO29) -> Net-(U2-GPIO28)
- U1 pad 1: Net-(U1-VCC) -> +3V3
- U10 pad 1: Net-(U10-VCC) -> +3V3
- U11 pad 1: Net-(U11-VCC) -> +3V3
- U2 pad 12: unconnected-(U2-GPIO13-Pad12) -> Net-(U2-GPIO13)
- U2 pad 13: unconnected-(U2-GPIO14-Pad13) -> Net-(U2-GPIO14)
- U2 pad 25: LRA_R -> Net-(U2-GPIO24)
- U2 pad 26: Net-(U2-GPIO25) -> LRA_R
- U2 pad 27: unconnected-(U2-GPIO26-Pad27) -> Net-(U2-GPIO26)
- U2 pad 28: unconnected-(U2-GPIO27-Pad28) -> Net-(U2-GPIO27)
- U2 pad 38: Net-(U2-GPIO30) -> unconnected-(U2-GPIO30-Pad38)
- U2 pad 48: unconnected-(U2-GPIO39-Pad48) -> Net-(U2-GPIO39)
- U2 pad 55: STICK_L_Y_OUT -> STICK_R_Y_OUT
- U2 pad 56: STICK_L_X_OUT -> STICK_R_X_OUT
- U2 pad 57: STICK_R_Y_OUT -> STICK_L_X_OUT
- U2 pad 58: STICK_R_X_OUT -> STICK_L_Y_OUT
- U3 pad 1: Net-(U3-VCC) -> +3V3
- U6 pad 1: Net-(U6-VCC) -> +3V3
- U7 pad 1: Net-(U7-VCC) -> +3V3
- U8 pad 1: Net-(U8-VCC) -> +3V3
- U9 pad 1: Net-(U9-VCC) -> +3V3
Routing:
- net Net-(U2-GPIO14): track 0.00 -> 57.9 mm, vias 0 -> 2
- net Net-(U2-GPIO24): track 0.00 -> 54.4 mm
- net Net-(U2-GPIO28): track 62.7 -> 8.91 mm
- net GRIP_R_BTN: track 8.36 -> 57.4 mm, vias 0 -> 2
- net STICK_R_X_OUT: track 0.00 -> 38.2 mm, vias 0 -> 2
- net STICK_R_Y_OUT: track 0.00 -> 38.2 mm, vias 0 -> 2
- net Net-(U2-GPIO13): track 0.00 -> 34.2 mm
- net Net-(U2-GPIO29): track 9.12 -> 41.3 mm
- net LRA_R: track 32.9 -> 58.1 mm, vias 0 -> 2
- net STICK_L_X_OUT: track 0.00 -> 22.0 mm, vias 0 -> 2
- net +3V3: track 34.4 -> 55.7 mm, vias 22 -> 33
- net STICK_L_Y_OUT: track 0.00 -> 21.0 mm, vias 0 -> 2
- net ABXY_EN: track 62.3 -> 79.7 mm
- net Net-(U2-GPIO27): track 0.00 -> 16.1 mm
- net Net-(U2-GPIO26): track 0.00 -> 15.9 mm
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- added copper zone on B.Cu, net +1V1

Commit message: Routing Updates
Parts:
- C1, C10, C11, C12, C13, C14, C19, C2, C23, C29, C30, C31, C32, C33, C34, C35, C36, C37, C38, C41, C9, D1, D2, D3, D4, D5, D6, Q1, Q2, R1, R10, R11, R5, R6, R7, R8, R9: moved to B.Cu
- moved Q2 161.9 mm to (122.8, 60.3), turned to -90 degrees
- moved C10 159.5 mm to (124.6, 58.0)
- moved C13 159.2 mm to (124.9, 59.1), turned to -90 degrees
- moved C14 155.9 mm to (121.5, 61.6), turned to 180 degrees
- moved D5 150.7 mm to (130.9, 61.6), turned to -45 degrees
- moved R6 150.2 mm to (124.9, 56.9), turned to 90 degrees
- moved R10 149.7 mm to (124.9, 60.6), turned to -90 degrees
- moved R8 148.6 mm to (123.8, 57.3), turned to 180 degrees
- moved D2 146.9 mm to (124.7, 62.1), turned to 180 degrees
- moved T3 145.2 mm to (125.2, 69.1)
- moved T4 142.0 mm to (122.9, 69.1)
- moved D6 139.8 mm to (120.0, 62.6), turned to -90 degrees
- moved J8 135.5 mm to (92.0, 46.6), turned to 90 degrees
- moved C25 124.6 mm to (93.9, 33.9), turned to 180 degrees
- moved C27 120.6 mm to (89.7, 34.4)
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Connections:
- J1 pad 1: LRA_R+ -> LRA_R-
- J1 pad 2: LRA_R- -> LRA_R+
Routing:
- net Net-(U2-RUN): track 5.80 -> 32.5 mm, vias 0 -> 3
- net LRA_L-: track 0.00 -> 23.4 mm
- net LRA_L+: track 0.00 -> 22.4 mm
- net LRA_R-: track 0.00 -> 21.8 mm
- net SWCLK: track 0.00 -> 20.9 mm, vias 0 -> 1
- net LRA_R+: track 0.00 -> 19.3 mm, vias 0 -> 2
- net SWD: track 0.00 -> 17.4 mm, vias 0 -> 1
- net GND: track 43.7 -> 54.6 mm, vias 26 -> 31
- net +1V1: track 10.2 -> 20.7 mm
- net Net-(C2-Pad1): track 0.00 -> 5.44 mm
- net /VREG_AVDD: track 0.00 -> 4.99 mm
- net XTAL_OUT: track 0.00 -> 4.62 mm
- net D-: track 29.7 -> 33.7 mm
- net D+: track 29.7 -> 33.8 mm
- net +3V3: track 55.7 -> 58.5 mm, vias 33 -> 37
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
Commit message: Routing updates
Routing:
- net +3V3: track 58.5 -> 373.9 mm, vias 37 -> 42
- net BTN_PWR: track 45.6 -> 56.7 mm
- net GND: track 54.6 -> 58.6 mm, vias 31 -> 36
- net STICK_R_Y_OUT: track 38.7 -> 40.3 mm, vias 3 -> 2
- net STICK_R_X_OUT: track 38.8 -> 40.1 mm
- net STICK_L_X_OUT: track 21.7 -> 22.4 mm
- added copper zone on B.Cu, net +3V3
- added copper zone on In2.Cu, net +3V3
- added copper zone on B.Cu, net GND
- added copper zone on F.Cu, net GND
- added copper zone on In1.Cu, net GND

Commit message: Routing updates
Parts:
- moved RGB10 6.81 mm to (42.4, 56.2)
- moved RGB11 6.81 mm to (47.2, 61.0)
- moved RGB12 6.81 mm to (52.0, 56.2)
- moved RGB9 6.81 mm to (47.2, 51.4)
- moved C38 0.13 mm to (80.5, 45.4)
- turned RGB5 to 180 degrees
- turned RGB6 to 180 degrees
- turned RGB7 to 180 degrees
- turned RGB8 to 180 degrees
Connections:
- SW3 pad 1: unconnected-(SW3-Pad1) -> GND
- SW4 pad 1: unconnected-(SW4-Pad1) -> GND
- SW5 pad 1: unconnected-(SW5-Pad1) -> GND
- SW6 pad 1: unconnected-(SW6-Pad1) -> GND
- SW7 pad 1: unconnected-(SW7-Pad1) -> GND
- SW8 pad 1: unconnected-(SW8-Pad1) -> GND
- U2 pad 81: unconnected-(U2-GND-Pad81) -> GND
Routing:
- net GND: track 58.6 -> 121.5 mm, vias 36 -> 44
- net STICK_R_RGB_OUT: track 0.00 -> 27.4 mm, vias 0 -> 2
- net RGB_DPAD_IN: track 1.13 -> 27.4 mm, vias 1 -> 2
- net Net-(RGB2-DOUT): track 2.46 -> 27.2 mm
- net STICK_L_RGB_IN: track 1.31 -> 24.0 mm
- net STICK_R_RGB_IN: track 1.26 -> 23.5 mm, vias 1 -> 2
- net Net-(RGB3-DOUT): track 2.41 -> 23.4 mm, vias 2 -> 3
- net Net-(RGB1-DOUT): track 2.32 -> 19.7 mm
- net +3V3: track 373.9 -> 356.6 mm, vias 42 -> 40
- net Net-(RGB10-DIN): track 2.53 -> 15.8 mm
- net Net-(RGB10-DOUT): track 2.37 -> 11.5 mm, vias 2 -> 3
- net unconnected-(SW7-Pad1): track 5.80 -> 0.00 mm
- net unconnected-(SW8-Pad1): track 5.80 -> 0.00 mm
- net unconnected-(SW6-Pad1): track 5.80 -> 0.00 mm
- net unconnected-(SW5-Pad1): track 5.80 -> 0.00 mm
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
Commit message: fun outline
Parts:
- added REF**: HHL_Logo, hhl:HHL_Logo, F.Cu at (26.7, 53.4)
- turned SW3 to 0 degrees
- turned SW4 to 0 degrees
Routing:
- net GRIP_R_BTN: track 57.8 -> 59.5 mm
- net GRIP_L_BTN: track 8.53 -> 10.2 mm
Other:
- board text added: "Latte Main PCB Designed by Mitch 11.2.2025"

Commit message: Routing updates
Parts:
- removed REF**: HHL_Logo, hhl:HHL_Logo
- moved R15 7.47 mm to (76.2, 31.6), turned to 90 degrees
Connections:
- R15 pad 1: Net-(R15-Pad1) -> Net-(U2-RUN)
- R15 pad 2: GND -> Net-(R15-Pad2)
- SW2 pad 1: Net-(R15-Pad1) -> GND
- SW2 pad 2: Net-(U2-RUN) -> Net-(R15-Pad2)
Routing:
- net Net-(R15-Pad2): track 0.00 -> 9.44 mm
- net Net-(R15-Pad1): track 7.67 -> 0.00 mm
- net Net-(U2-RUN): track 33.0 -> 25.6 mm
- net GND: track 121.2 -> 126.9 mm

Commit message: Prod 1
Parts:
- added REF**: HHL_Logo, hhl:HHL_Logo, F.Cu at (27.1, 53.3)
Routing:
- net GND: track 126.9 -> 122.4 mm
