File: PCB/Projects/Main Board/Latte_Main_Board.kicad_pcb (KiCad board)
At the start: 4 copper layers, 114 x 50.5 mm, 121 parts, among them J1 SM02B-SURS-TF_LF__SN_, J2 SM02B-SURS-TF_LF__SN_, J3 Molex 505110-0892, J4 Molex 505110-0592, J5 Molex 505110-0892, J6 Molex 505110-0592, J8 Conn_01x04_Pin, J9 Molex 505110-1792, Q1 MMBT2222A, Q2 MMBT2222A, SW1 SW_Push, SW2 SW_Push, SW3 SW_Push, SW4 SW_Push, SW5 SW_Push, SW6 SW_Push, SW7 SW_Push, SW8 SW_Push, SW9 1TS026A-1000-0550, U1 HAL4395, U10 HAL4395, U11 HAL4395, U2 RP2350_80QFN, U3 HAL4395, U4 ST_LSM6, U5 ST_LSM6, U6 HAL4395, U7 HAL4395, U8 HAL4395, U9 HAL4395, Y1 ABM8-272-T3

Commit message: Updates
Connections:
- C1 pad 2: GND -> STICK_L_BTN_OUT
- C10 pad 2: GND -> STICK_L_BTN_OUT
- C11 pad 1: GND -> STICK_L_BTN_OUT
- C12 pad 2: GND -> STICK_L_BTN_OUT
- C13 pad 1: GND -> STICK_L_BTN_OUT
- C14 pad 2: GND -> STICK_L_BTN_OUT
- C17 pad 2: GND -> STICK_L_BTN_OUT
- C18 pad 2: GND -> STICK_L_BTN_OUT
- C19 pad 2: GND -> STICK_L_BTN_OUT
- C2 pad 2: GND -> STICK_L_BTN_OUT
- C23 pad 2: GND -> STICK_L_BTN_OUT
- C24 pad 1: GND -> STICK_L_BTN_OUT
- C25 pad 1: GND -> STICK_L_BTN_OUT
- C26 pad 1: GND -> STICK_L_BTN_OUT
- C27 pad 1: GND -> STICK_L_BTN_OUT
- C29 pad 2: GND -> STICK_L_BTN_OUT
- C3 pad 2: GND -> STICK_L_BTN_OUT
- C30 pad 2: GND -> STICK_L_BTN_OUT
- C31 pad 2: GND -> STICK_L_BTN_OUT
- C32 pad 2: GND -> STICK_L_BTN_OUT
- C33 pad 2: GND -> STICK_L_BTN_OUT
- C34 pad 2: GND -> STICK_L_BTN_OUT
- C35 pad 2: GND -> STICK_L_BTN_OUT
- C36 pad 2: GND -> STICK_L_BTN_OUT
- C37 pad 2: GND -> STICK_L_BTN_OUT
- C38 pad 2: GND -> STICK_L_BTN_OUT
- C39 pad 2: GND -> STICK_L_BTN_OUT
- C4 pad 2: GND -> STICK_L_BTN_OUT
- C40 pad 2: GND -> STICK_L_BTN_OUT
- C41 pad 2: GND -> STICK_L_BTN_OUT
- C5 pad 2: GND -> STICK_L_BTN_OUT
- C6 pad 2: GND -> STICK_L_BTN_OUT
- C7 pad 2: GND -> STICK_L_BTN_OUT
- C8 pad 2: GND -> STICK_L_BTN_OUT
- C9 pad 2: GND -> STICK_L_BTN_OUT
- D1 pad 2: GND -> STICK_L_BTN_OUT
- D2 pad 2: GND -> STICK_L_BTN_OUT
- D4 pad 2: GND -> STICK_L_BTN_OUT
- D6 pad 2: GND -> STICK_L_BTN_OUT
- J1 pad S1: GND -> STICK_L_BTN_OUT
- J1 pad S2: GND -> STICK_L_BTN_OUT
- J2 pad S1: GND -> STICK_L_BTN_OUT
- J2 pad S2: GND -> STICK_L_BTN_OUT
- J3 pad 4: GND -> STICK_L_BTN_OUT
- J3 pad 8: STICK_R_BTN_OUT -> STICK_L_BTN_OUT
- J4 pad 5: GND -> STICK_L_BTN_OUT
- J5 pad 4: GND -> STICK_L_BTN_OUT
- J6 pad 5: GND -> STICK_L_BTN_OUT
- J8 pad 3: GND -> STICK_L_BTN_OUT
- J9 pad 11: GND -> STICK_L_BTN_OUT
- J9 pad 12: GND -> STICK_L_BTN_OUT
- Q1 pad 2: GND -> STICK_L_BTN_OUT
- Q2 pad 2: GND -> STICK_L_BTN_OUT
- R5 pad 1: GND -> STICK_L_BTN_OUT
- R6 pad 1: GND -> STICK_L_BTN_OUT
- RGB1 pad 4: GND -> STICK_L_BTN_OUT
- RGB10 pad 4: GND -> STICK_L_BTN_OUT
- RGB11 pad 4: GND -> STICK_L_BTN_OUT
- RGB12 pad 4: GND -> STICK_L_BTN_OUT
- RGB2 pad 4: GND -> STICK_L_BTN_OUT
- RGB3 pad 4: GND -> STICK_L_BTN_OUT
- RGB4 pad 4: GND -> STICK_L_BTN_OUT
- RGB5 pad 4: GND -> STICK_L_BTN_OUT
- RGB6 pad 4: GND -> STICK_L_BTN_OUT
- RGB7 pad 4: GND -> STICK_L_BTN_OUT
- RGB8 pad 4: GND -> STICK_L_BTN_OUT
- RGB9 pad 4: GND -> STICK_L_BTN_OUT
- SW1 pad 1: GND -> STICK_L_BTN_OUT
- SW2 pad 1: GND -> STICK_L_BTN_OUT
- SW3 pad 1: GND -> STICK_L_BTN_OUT
- SW4 pad 1: GND -> STICK_L_BTN_OUT
- SW5 pad 1: GND -> STICK_L_BTN_OUT
- SW6 pad 1: GND -> STICK_L_BTN_OUT
- SW7 pad 1: GND -> STICK_L_BTN_OUT
- SW8 pad 1: GND -> STICK_L_BTN_OUT
- SW9 pad 1: GND -> STICK_L_BTN_OUT
- SW9 pad 2: GND -> STICK_L_BTN_OUT
- U1 pad 3: GND -> STICK_L_BTN_OUT
- U10 pad 3: GND -> STICK_L_BTN_OUT
- U11 pad 3: GND -> STICK_L_BTN_OUT
- U2 pad 62: GND -> STICK_L_BTN_OUT
- U2 pad 81: GND -> STICK_L_BTN_OUT
- U3 pad 3: GND -> STICK_L_BTN_OUT
- U4 pad 2: GND -> STICK_L_BTN_OUT
- U4 pad 3: GND -> STICK_L_BTN_OUT
- U4 pad 6: GND -> STICK_L_BTN_OUT
- U4 pad 7: GND -> STICK_L_BTN_OUT
- U5 pad 2: GND -> STICK_L_BTN_OUT
- U5 pad 3: GND -> STICK_L_BTN_OUT
- U5 pad 6: GND -> STICK_L_BTN_OUT
- U5 pad 7: GND -> STICK_L_BTN_OUT
- U6 pad 3: GND -> STICK_L_BTN_OUT
- U7 pad 3: GND -> STICK_L_BTN_OUT
- U8 pad 3: GND -> STICK_L_BTN_OUT
- U9 pad 3: GND -> STICK_L_BTN_OUT
- Y1 pad 2: GND -> STICK_L_BTN_OUT
- Y1 pad 4: GND -> STICK_L_BTN_OUT
Routing:
- net STICK_L_BTN_OUT: track 0.00 -> 123.0 mm, vias 0 -> 43
- net GND: track 123.0 -> 0.00 mm, vias 43 -> 0
- added copper zone on B.Cu, net STICK_L_BTN_OUT
- added copper zone on F.Cu, net STICK_L_BTN_OUT
- added copper zone on In1.Cu, net STICK_L_BTN_OUT
- removed copper zone on B.Cu, net GND
- removed copper zone on F.Cu, net GND
- removed copper zone on In1.Cu, net GND
