File: PCB/Projects/Main Board/Latte_Main_Board.kicad_sch (KiCad schematic)
At the start: 120 parts, among them J1 SM02B-SURS-TF_LF__SN_, J2 SM02B-SURS-TF_LF__SN_, J3 Molex 505110-0892, J4 Molex 505110-0592, J5 Molex 505110-0892, J6 Molex 505110-0592, J8 Conn_01x04_Pin, J9 Molex 505110-1792, Q1 MMBT2222A, Q2 MMBT2222A, SW1 SW_Push, SW2 SW_Push, SW3 SW_Push, SW4 SW_Push, SW5 SW_Push, SW6 SW_Push, SW7 SW_Push, SW8 SW_Push, SW9 1TS026A-1000-0550, U1 HAL4395, U10 HAL4395, U11 HAL4395, U2 RP2350_80QFN, U3 HAL4395, U4 ST_LSM6, U5 ST_LSM6, U6 HAL4395, U7 HAL4395, U8 HAL4395, U9 HAL4395, Y1 ABM8-272-T3

Commit message: Updates
Connections:
- net STICK_L_BTN_OUT is gone; now on net GND: J5.8 (Pin_8)
- net STICK_R_BTN_OUT is gone; now on net GND: J3.8 (Pin_8)
Changed lines of the file:
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@@
 	)
 	(junction
+		(at 25.4 252.73)
+		(diameter 0)
+		(color 0 0 0 0)
+	)
+	(junction
 		(at 15.24 123.19)
 		(diameter 0)
@@
 	)
 	(junction
+		(at 25.4 278.13)
+		(diameter 0)
+		(color 0 0 0 0)
+	)
+	(junction
 		(at 250.19 46.99)
 		(diameter 0)
@@
 	(wire
 		(pts
-			(xy 24.13 252.73) (xy 26.67 252.73)
+			(xy 24.13 252.73) (xy 25.4 252.73)
 		)
 		(stroke
@@
 	(wire
 		(pts
+			(xy 25.4 252.73) (xy 26.67 252.73)
+		)
+		(stroke
+			(width 0)
+			(type default)
+		)
+	)
+	(wire
+		(pts
 			(xy 143.51 205.74) (xy 142.24 205.74)
 		)
@@
 	(wire
 		(pts
+			(xy 25.4 278.13) (xy 26.67 278.13)
+		)
+		(stroke
+			(width 0)
+			(type default)
+		)
+	)
+	(wire
+		(pts
 			(xy 372.11 181.61) (xy 368.3 181.61)
 		)
@@
 	(wire
 		(pts
-			(xy 24.13 278.13) (xy 26.67 278.13)
+			(xy 24.13 278.13) (xy 25.4 278.13)
 		)
 		(stroke
@@
 	)
 	(symbol
+		(lib_id "power:GND")
+		(at 25.4 278.13 0)
+		(unit 1)
+		(exclude_from_sim no)
+		(in_bom yes)
+		(on_board yes)
+		(dnp no)
+		(property "Reference" "#PWR094"
+			(at 25.4 284.48 0)
+			(effects
+				(font
+					(size 1.27 1.27)
+				)
+				(hide yes)
+			)
+		)
+		(property "Value" "GND"
+			(at 25.4 283.21 90)
+			(effects
+				(font
+					(size 1.27 1.27)
+				)
+			)
+		)
+		(property "Footprint" ""
+			(at 25.4 278.13 0)
+			(effects
+				(font
+					(size 1.27 1.27)
+				)
+				(hide yes)
+			)
+		)
+		(property "Datasheet" ""
+			(at 25.4 278.13 0)
+			(effects
+				(font
+					(size 1.27 1.27)
+				)
+				(hide yes)
+			)
+		)
+		(property "Description" "Power symbol creates a global label with name \"GND\" , ground"
+			(at 25.4 278.13 0)
+			(effects
+				(font
+					(size 1.27 1.27)
+				)
+				(hide yes)
+			)
+		)
+		(pin "1"
+		)
+		(instances
+			(project "Latte_Main_Board"
+				(path "/e225eb3e-e7d7-4a30-a02a-c99a852af5d1"
+					(reference "#PWR094")
+					(unit 1)
+				)
+			)
+		)
+	)
+	(symbol
 		(lib_id "Device:R")
 		(at 241.3 53.34 180)
@@
 					(unit 1)
 				)
+			)
+		)
+	)
+	(symbol
+		(lib_id "power:GND")
+		(at 25.4 252.73 0)
+		(unit 1)
+		(exclude_from_sim no)
+		(in_bom yes)
+		(on_board yes)
+		(dnp no)
+		(property "Reference" "#PWR093"
+			(at 25.4 259.08 0)
+			(effects
+				(font
+					(size 1.27 1.27)
+				)
+				(hide yes)
+			)
+		)
+		(property "Value" "GND"
+			(at 25.4 257.81 90)
+			(effects
+				(font
+					(size 1.27 1.27)
+				)
+			)
+		)
+		(property "Footprint" ""
+			(at 25.4 252.73 0)
+			(effects
+				(font
+					(size 1.27 1.27)
+				)
+				(hide yes)
+			)
+		)
+		(property "Datasheet" ""
+			(at 25.4 252.73 0)
+			(effects
+				(font
+					(size 1.27 1.27)
+				)
+				(hide yes)
+			)
+		)
+		(property "Description" "Power symbol creates a global label with name \"GND\" , ground"
+			(at 25.4 252.73 0)
+			(effects
+				(font
+					(size 1.27 1.27)
+				)
+				(hide yes)
+			)
+		)
+		(pin "1"
+		)
+		(instances
+			(project "Latte_Main_Board"
+				(path "/e225eb3e-e7d7-4a30-a02a-c99a852af5d1"
+					(reference "#PWR093")
+					(unit 1)
+				)
