File: PCB/Projects/Trigger FPC/FPC_Trigger_Board.kicad_pcb (KiCad board)
At the start: 2 copper layers, 127.6 x 29.7 mm, 10 parts, among them J1 Conn_01x05_Pin, J2 Conn_01x05_Pin, U1 HAL4395, U2 HAL4395, U3 HAL4395, U4 HAL4395

Commit message: Prod 1
Parts:
- moved C1 1.06 mm to (270.4, 156.4)

Commit message: FPC Fixes
Parts:
- U1, U2, U3, U4: footprint Package_TO_SOT_SMD:SOT-23-5 -> hhl:SOT-23-5L
- moved U1 5.00 mm to (272.1, 154.2), turned to 90 degrees
- moved U3 5.00 mm to (165.3, 154.2)
- moved C1 4.76 mm to (271.5, 151.8), turned to 180 degrees
- moved C3 3.22 mm to (166.9, 156.7), turned to 180 degrees
- turned U2 to -90 degrees
- turned U4 to -90 degrees
Connections:
- U1 pad 2: GNDL -> TRIGGER_EN_L
- U1 pad 3: TRIGGER_EN_L -> GNDL
- U2 pad 2: GNDL -> TRIGGER_EN_L
- U2 pad 3: TRIGGER_EN_L -> GNDL
- U3 pad 2: GND -> TRIGGER_EN_R
- U3 pad 3: TRIGGER_EN_R -> GND
- U4 pad 2: GND -> TRIGGER_EN_R
- U4 pad 3: TRIGGER_EN_R -> GND
Routing:
- net GND: track 3.99 -> 66.3 mm, vias 4 -> 8
- net ADC_1: track 83.4 -> 71.7 mm
- net GNDL: track 19.5 -> 10.9 mm, vias 5 -> 8
- net ADC_3: track 84.7 -> 77.0 mm
- net +3V3L: track 90.9 -> 83.7 mm
- net TRIGGER_EN_R: track 91.1 -> 86.3 mm
- net TRIGGER_EN_L: track 85.5 -> 80.9 mm
- net +3V3: track 86.6 -> 89.4 mm
Other:
- outline, holes or cut-outs redrawn
