File: PCB/Projects/Trigger FPC/FPC_Trigger_Board.kicad_sch (KiCad schematic)
At the start: 10 parts, among them J1 Conn_01x05_Pin, J2 Conn_01x05_Pin, U1 HAL4395, U2 HAL4395, U3 HAL4395, U4 HAL4395

Commit message: Prod 1
Parts:
- C1, C2, C3, C4: LCSC (none) -> C76934; MPN (none) -> GRM033R61A104KE15D; Manufacturer (none) -> muRata
- J1, J2: now not fitted
- U1, U2, U3, U4: LCSC (none) -> C49165022; MPN (none) -> HAL4395SO5; Manufacturer (none) -> Hallwee

Commit message: FPC Fixes
Parts:
- removed U1, U2, U3, U4: HAL4395, Package_TO_SOT_SMD:SOT-23-5, symbol hhl:HAL4395SO5
- added U1, U2, U3, U4: HAL4395, hhl:SOT-23-5L, symbol Regulator_Linear:TLV70012_SOT23-5
Connections:
- net +3V3: now also U3.1 (VCC), U4.1 (VCC)
- net +3V3L: now also U1.1 (VCC), U2.1 (VCC)
- net ADC_0: now also U4.5 (OUT)
- net ADC_1: now also U3.5 (OUT)
- net ADC_2: now also U2.5 (OUT)
- net ADC_3: now also U1.5 (OUT)
- net GND: now also U3.3 (GND), U4.3 (GND)
- net GNDL: now also U1.3 (GND), U2.3 (GND)
- net TRIGGER_EN_L: now also U1.2 (~{EN}), U2.2 (~{EN})
- net TRIGGER_EN_R: now also U3.2 (~{EN}), U4.2 (~{EN})
